Commit message: Add new robot assets and trainig configurations for the X2 29DOF robot.

File: src/holosoma/holosoma/data/robots/x2/x2_29dof.urdf (robot description, URDF)
Before this commit: robot x2t2.5, 39 links, 38 joints
Links:
- added link LL_FOOT, mass 1e-9; visual box size=0.001 0.001 0.001
- added link LR_FOOT, mass 1e-9; visual box size=0.001 0.001 0.001
- added link imu_in_pelvis; visual box size=0.001 0.001 0.001
- added link left_foot_contact_point, mass 0.001; visual box size=0.001 0.001 0.001
- added link lidar_chest_front; visual box size=0.001 0.001 0.001
- added link right_foot_contact_point, mass 0.001; visual box size=0.001 0.001 0.001
Joints:
- added joint LL_FOOT_frame: type fixed, parent left_ankle_roll_link, child LL_FOOT, origin xyz=0.0037 0 -0.073 rpy=0 0 0
- added joint LR_FOOT_frame: type fixed, parent right_ankle_roll_link, child LR_FOOT, origin xyz=0.037 0 -0.073 rpy=0 0 0
- added joint imu_in_pelvis_compat_joint: type fixed, parent pelvis, child imu_in_pelvis, origin xyz=0.0239464627920677 -0.00022868187247424 0.0417100000000296 rpy=0 0 0
- added joint left_foot_contact_point: type fixed, parent left_ankle_roll_link, child left_foot_contact_point, origin xyz=0.037 0 -0.073 rpy=0 0 0
- added joint lidar_chest_front_joint: type fixed, parent torso_link, child lidar_chest_front, origin xyz=0.102633 0 0.181587 rpy=-1.570796 0 0
- added joint right_foot_contact_point: type fixed, parent right_ankle_roll_link, child right_foot_contact_point, origin xyz=0.037 0 -0.073 rpy=0 0 0
- joint head_pitch_joint: axis 0 1 0 -> (none); limit lower=-0.3838 upper=0.3838 effort=0.6 velocity=6.28 -> (none)
- joint head_yaw_joint: axis 0 0 1 -> (none); limit lower=-0.366 upper=0.366 effort=2.6 velocity=6.019 -> (none)
- joint left_elbow_joint: type fixed -> revolute
- joint left_shoulder_pitch_joint: type fixed -> revolute
- joint left_shoulder_roll_joint: type fixed -> revolute
- joint left_shoulder_yaw_joint: type fixed -> revolute
- joint left_wrist_pitch_joint: type fixed -> revolute
- joint left_wrist_roll_joint: type fixed -> revolute
- joint left_wrist_yaw_joint: type fixed -> revolute
- joint right_elbow_joint: type fixed -> revolute
- joint right_shoulder_pitch_joint: type fixed -> revolute
- joint right_shoulder_roll_joint: type fixed -> revolute
- joint right_shoulder_yaw_joint: type fixed -> revolute
- joint right_wrist_pitch_joint: type fixed -> revolute
- joint right_wrist_roll_joint: type fixed -> revolute
- joint right_wrist_yaw_joint: type fixed -> revolute
- joint waist_pitch_joint: type fixed -> revolute
- joint waist_roll_joint: type fixed -> revolute
- joint waist_yaw_joint: type fixed -> revolute
